Commit message: ATI GAMMA sensor added in urdf and MoveIt! configuration

File: fetch_description/robots/fetch.urdf (robot description, URDF)
Before this commit: robot fetch, 26 links, 25 joints
Links:
- added link ati_link, mass 0.255; collision cylinder length=0.0333 radius=0.058; visual cylinder length=0.0333 radius=0.0377
Joints:
- added joint ati_axis: type fixed, parent wrist_roll_link, child ati_link, origin xyz=${0.0190+0.0333} 0 0 rpy=0.894 0 0, axis 0 0 0
- joint gripper_axis: origin xyz=0.16645 0 0 rpy=0 0 0 -> xyz=${0.16645-0.019} 0 0 rpy=0 0 0; parent wrist_roll_link -> ati_link

Commit message: Updated fetch_telop

File: fetch_description/robots/fetch.urdf (robot description, URDF)
Before this commit: robot fetch, 27 links, 26 joints
Joints:
- joint wrist_roll_joint: limit effort=7.36 velocity=2.268 -> lower=-3.16 upper=3.16 effort=7.36 velocity=2.268; type continuous -> revolute

Commit message: New sensor.stl and new fingers applied to .urdf

File: fetch_description/robots/fetch.urdf (robot description, URDF)
Before this commit: robot fetch, 27 links, 26 joints
Links:
- added link EoF_link
- link ati_link: geometry collision cylinder length=0.0333 radius=0.063; visual mesh filename=package://fetch_description/meshes/ati_sensor.stl
- link l_gripper_finger_link: geometry collision mesh filename=package://fetch_description/meshes/fingers/simplified_1/l_f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; visual mesh filename=package://fetch_description/meshes/fingers/simplified_1/l_f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
- link r_gripper_finger_link: geometry collision mesh filename=package://fetch_description/meshes/fingers/simplified_1/r_f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; visual mesh filename=package://fetch_description/meshes/fingers/simplified_1/r_f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
Joints:
- added joint EoF_axis: type fixed, parent gripper_link, child EoF_link, origin xyz=0.10 0 0 rpy=0 0 0
- joint forearm_roll_joint: limit effort=29.35 velocity=1.571 -> lower=-3.05 upper=3.05 effort=29.35 velocity=1.571; type continuous -> revolute
- joint upperarm_roll_joint: limit effort=76.94 velocity=1.571 -> lower=-3.05 upper=3.05 effort=76.94 velocity=1.571; type continuous -> revolute
- joint wrist_roll_joint: limit lower=-3.16 upper=3.16 effort=7.36 velocity=2.268 -> lower=-3.05 upper=3.05 effort=7.36 velocity=2.268
