Commit message: Calibration and urdf update

File: fetch_description/robots/calibrated/calibrated_2024_12_09_20_00_06.urdf (robot description, URDF)
Before this commit: robot fetch, 28 links, 27 joints
Links:
- removed link EoF_link
- added link finger_tip_link
- link l_gripper_finger_link: geometry collision mesh filename=package://fetch_description/meshes/fingers/simplified_1/l_f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; visual mesh filename=package://fetch_description/meshes/fingers/simplified_1/l_f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
- link r_gripper_finger_link: geometry collision mesh filename=package://fetch_description/meshes/fingers/simplified_1/r_f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; visual mesh filename=package://fetch_description/meshes/fingers/simplified_1/r_f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
Joints:
- removed joint EoF_axis
- added joint finger_tip_axis: type fixed, parent gripper_link, child finger_tip_link, origin xyz=0.10 0 0 rpy=0 0 0
- joint ati_axis: origin xyz=${0.0190+0.0333} 0 0 rpy=0.894 0 0 -> xyz=0.0523 0 0 rpy=-0.8287 0 0
- joint gripper_axis: origin xyz=${0.16645-0.019} 0 0 rpy=0 0 0 -> xyz=0.14745 0 0 rpy=0 0 0
- joint head_camera_rgb_joint: origin xyz=0 0.02 0 rpy=0 0 0 -> xyz=-0.00407983 0.02177149 -0.00387805 rpy=-0.00779133 -0.00013198 -0.00269151
- joint head_pan_joint: origin xyz=0.053125 0 0.603001417713939 rpy=0 0 0 -> xyz=0.05527368 0.00042896 0.61020700 rpy=0.00121442 0.00430826 0.00441649

File: fetch_description/robots/calibrated/calibrated_2024_12_09_20_00_06_original_fingers.urdf (robot description, URDF)
Before this commit: robot fetch, 28 links, 27 joints
Links:
- removed link EoF_link
- added link finger_tip_link
- link l_gripper_finger_link: geometry collision mesh filename=package://fetch_description/meshes/l_gripper_finger_link.STL; visual mesh filename=package://fetch_description/meshes/l_gripper_finger_link.STL
- link r_gripper_finger_link: geometry collision mesh filename=package://fetch_description/meshes/r_gripper_finger_link.STL; visual mesh filename=package://fetch_description/meshes/r_gripper_finger_link.STL
Joints:
- removed joint EoF_axis
- added joint finger_tip_axis: type fixed, parent gripper_link, child finger_tip_link, origin xyz=0.03 0 0 rpy=0 0 0
- joint ati_axis: origin xyz=${0.0190+0.0333} 0 0 rpy=0.894 0 0 -> xyz=0.0523 0 0 rpy=-0.8287 0 0
- joint gripper_axis: origin xyz=${0.16645-0.019} 0 0 rpy=0 0 0 -> xyz=0.14745 0 0 rpy=0 0 0
- joint head_camera_rgb_joint: origin xyz=0 0.02 0 rpy=0 0 0 -> xyz=-0.00407983 0.02177149 -0.00387805 rpy=-0.00779133 -0.00013198 -0.00269151
- joint head_pan_joint: origin xyz=0.053125 0 0.603001417713939 rpy=0 0 0 -> xyz=0.05527368 0.00042896 0.61020700 rpy=0.00121442 0.00430826 0.00441649

File: fetch_description/robots/fetch_original_fingers.urdf (robot description, URDF)
Before this commit: robot fetch, 28 links, 27 joints
Links:
- link l_gripper_finger_link: geometry collision mesh filename=package://fetch_description/meshes/l_gripper_finger_link.STL; visual mesh filename=package://fetch_description/meshes/l_gripper_finger_link.STL
- link r_gripper_finger_link: geometry collision mesh filename=package://fetch_description/meshes/r_gripper_finger_link.STL; visual mesh filename=package://fetch_description/meshes/r_gripper_finger_link.STL
Joints:
- joint finger_tip_axis: origin xyz=0.10 0 0 rpy=0 0 0 -> xyz=0.03 0 0 rpy=0 0 0
